File: First_Distortion_FD-1.kicad_pcb (KiCad board)
At the start: 2 copper layers, 54 x 73.5 mm, 39 parts, among them X1 DC_Jack_PCB, X2 DC_Jack_Wire, X3 Battery_Conn, X4 CON

Commit message: Добавление чертежа развёртки корпуса для сверления
Parts:
- added REF**: Hammond_1590B, Alimach:Hammond_1590B, F.Cu at (-68.2, 71.0)
- moved ? 21.2 mm to (129.5, 85.0)
- moved C1 21.2 mm to (129.0, 142.0)
- moved C2 21.2 mm to (136.0, 114.5)
- moved C3 21.2 mm to (110.0, 111.0)
- moved C4 21.2 mm to (121.5, 102.0)
- moved C5 21.2 mm to (100.5, 94.5)
- moved C6 21.2 mm to (134.5, 110.0)
- moved C7 21.2 mm to (97.0, 97.0)
- moved C8 21.2 mm to (118.0, 99.0)
- moved C9 21.2 mm to (123.5, 114.5)
- moved DA1 21.2 mm to (107.5, 107.0)
- moved G*** 21.2 mm to (93.0, 87.5)
- moved G*** 21.2 mm to (133.5, 149.0)
- moved R1 21.2 mm to (127.4, 138.5)
- moved R10 21.2 mm to (104.5, 107.5)
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Other:
- board text added: "0"
- board text added: "Развёртка корпуса"
